Commit message: Updating livox_mid70 xacro to enable mounting
- Updated to enable mounting on joints in other URDFs
- Fixed (?) issue with frames, so that the cloud data has the same frame
as the sensor name

File: urdf/livox_mid70.xacro (robot description, xacro)
@@ -6,5 +6,4 @@
   <xacro:property name="horizontal_fov" value="70.4"/>
   <xacro:property name="vertical_fov" value="70.4"/>
-  <xacro:property name="ros_topic" value="scan"/>
   <xacro:property name="samples" value="10000"/>
   <xacro:property name="downsample" value="1"/>
@@ -17,11 +16,11 @@
     </inertial>
   </xacro:macro>
-  <xacro:macro name="Livox_Mid_gazebo_sensor" params="visualize:=True update_rate:=10 resolution:=0.002 noise_mean:=0.0 noise_stddev:=0.01 name:=livox">
+  <xacro:macro name="Livox_Mid_gazebo_sensor" params="visualize:=True update_rate:=10 resolution:=0.002 noise_mean:=0.0 noise_stddev:=0.01 name:=livox topic:=pointcloud">
     <gazebo reference="${name}">
-      <sensor type="ray" name="laser_${name}">
+      <sensor type="ray" name="${name}">
         <pose>0 0 0 0 0 0</pose>
         <visualize>${visualize}</visualize>
         <update_rate>${update_rate}</update_rate>
-        <!-- This ray plgin is only for visualization. -->
+        <!-- This ray pulgin is only for visualization. -->
         <plugin name="gazebo_ros_laser_controller" filename="liblivox_laser_simulation.so">
 			<ray>
@@ -55,17 +54,21 @@
 		  <downsample>${downsample}</downsample>
 		  <csv_file_name>package://livox_laser_simulation/scan_mode/mid70.csv</csv_file_name>
-		  <ros_topic>${ros_topic}</ros_topic>
+		  <ros_topic>${topic}</ros_topic>
         </plugin>
       </sensor>
     </gazebo>
   </xacro:macro>
-  <xacro:macro name="Livox_Mid70" params="visualize:=True name:=livox">
+  <xacro:macro name="Livox_Mid70" params="*origin visualize:=True name:=livox topic=pointcloud parent=base_link">
+		<joint name="${name}_base_mount_joint" type="fixed">
+			<xacro:insert_block name="origin" />
+			<parent link="${parent}" />
+			<child link="${name}_base" />
+		</joint>
     <link name="${name}_base">
       <xacro:null_inertial/>
       <visual>
-        <origin xyz="0.00 0 0.00" rpy="0 0 0"/>
+				<origin xyz="0 0 0" rpy="0 0 0" />
         <geometry>
-          <mesh filename="package://livox_laser_simulation/meshes/livox_mid40.dae">
-          </mesh>
+          <mesh filename="package://livox_laser_simulation/meshes/livox_mid40.dae"/>
         </geometry>
       </visual>
@@ -73,6 +76,5 @@
           <origin xyz="0 0 0" rpy="0 0 0" />
           <geometry>
-          <mesh filename="package://livox_laser_simulation/meshes/livox_mid40.dae">
-          </mesh>
+            <mesh filename="package://livox_laser_simulation/meshes/livox_mid40.dae"/>
           </geometry>
       </collision>
@@ -86,8 +88,5 @@
       <origin rpy="0 0 0" xyz="0.0 0.0 0.0"/>
     </joint>
-    <xacro:Livox_Mid_gazebo_sensor name="${name}" visualize="${visualize}"/>
+    <xacro:Livox_Mid_gazebo_sensor name="${name}" visualize="${visualize}" topic="${topic}"/>
   </xacro:macro>
-    <xacro:Livox_Mid70 name="livox"/>
-  <xacro:include filename="$(find livox_laser_simulation)/urdf/standardrobots_oasis300.xacro"/>
-  <xacro:link_oasis name="oasis"/>
 </robot>
